Commit message: Current progress
Excluding logic and turtlesim parts

File: description/camera.xacro (robot description, xacro)
@@ -12,5 +12,5 @@
         <parent link="chassis"/>
         <child link="camera"/>
-        <origin xyz="${(chassis_length-cam_thickness)/2} 0 ${(chassis_height+cam_height)/2}" rpy="0 0 0"/>
+        <origin xyz="${(chassis_length+cam_thickness)/2} 0 ${(chassis_height-cam_height)/2}" rpy="0 0 0"/> <!-- ${(chassis_height+cam_height)/2} -->
     </joint>
     <link name="camera">
@@ -41,5 +41,5 @@
             <update_rate>10</update_rate>
             <camera>
-                <horizontal_fov>1.089</horizontal_fov> <!-- in radians -->
+                <horizontal_fov>1.089</horizontal_fov> <!-- 1.089 in radians -->
                 <image>
                     <format>R8G8B8</format>

File: description/car.xacro (robot description, xacro)
@@ -12,6 +12,24 @@
         <color rgba="1 1 1 1"/>
     </material>
+    <material name="red">
+        <color rgba="1 0 0 1"/>
+    </material>
+    <material name="yellow">
+        <color rgba="1 1 0 1"/>
+    </material>
     <link name="base_link">
     </link>
+    <joint name="base_footprint_joint" type="fixed">
+        <parent link="base_link"/>
+        <child link="base_footprint"/>
+        <origin xyz="0 0 0" rpy="0 0 0"/>
+    </joint>
+    <link name="base_footprint">
+    </link>
+    <joint name="chassis_joint" type="fixed">
+        <origin xyz="0 0 ${wheel_radius+chassis_height/2}" />
+        <parent link="base_link"/>
+        <child link="chassis"/>
+    </joint>
     <link name="chassis">
         <visual>
@@ -34,9 +52,4 @@
         <material>Gazebo/White</material>
     </gazebo>
-    <joint name="chassis_joint" type="fixed">
-        <origin xyz="0 0 ${wheel_radius+chassis_height/2}" />
-        <parent link="base_link"/>
-        <child link="chassis"/>
-    </joint>
     <link name="left_front_wheel">
         <visual>

File: description/robot_car.urdf.xacro (robot description, xacro)
@@ -10,4 +10,6 @@
         <xacro:include filename="gazebo_control.xacro" />
     </xacro:unless>
+    <!-- <xacro:include filename="lidar.xacro"/> -->
     <xacro:include filename="camera.xacro"/>
+    <xacro:include filename="marker.xacro"/>
 </robot>
